File: elettronica/main.brd (EAGLE design)
At the start: 100 x 80 mm, 91 parts, among them IC1 7805T, IC2 7805T, IC3 74LS595D, J2 455-1750-1-ND, SW2 EC12E_SW

Commit message: aggiunta la motor hub
Parts:
- removed B1: ARDUINO_MEGA_R3FULL, SparkFun-Boards:ARDUINO_MEGA
- removed C1, C3: 0.1uF, SparkFun-Capacitors:CAP-PTH-SMALL-KIT
- removed C2, C4: 0.22uF, SparkFun-Capacitors:CAP-PTH-SMALL-KIT
- removed C7, C8: (no value), rcl:C1206
- removed D1, D3: 1N4148, diode:DO35-7
- removed DISPLAY1: DISPLAY128X128, Display 128x128:DISPLAY128X128
- removed IC3: 74LS595D, 74xx-us:SO16
- removed LED1, LED10, LED11, LED12, LED13, LED14, LED2, LED9: TLLG4400, led:LED3MM
- removed LED7, LED8: TLLR4400, led:LED3MM
- removed M1: (no value), mfrc522-module:RFID-RC522
- removed R12: 330, eagle-ltspice:R1206
- removed R13: 10k, eagle-ltspice:R1206
- removed R14: (no value), rcl:M1206
- removed R15: 100, eagle-ltspice:R1206
- removed R20: 20k, eagle-ltspice:0204/7
- removed R21: 10k, eagle-ltspice:0204/7
- removed RN1: 330, resistor-net:RN-8
- removed SV1, SV2, SV3: (no value), con-lstb:MA03-2
- removed SW2: EC12E_SW, switch-alps:ALPS_EC12E_SW
- removed U$1, U$12, U$13, U$2: DRILL_SWITCH, Switch drill:DRILL_SWITCH
- removed U$10, U$11, U$14, U$9: VHN5019, VHN5019:MOTOR-SHIELD
- removed U$15: BNO055, BNO055:BNO005
- removed U$16: HC-05, HC-05:HC-05
- removed X1, X5: (no value), con-ptr500:AK500/2-H
- added D11, D12, D13, D14, D15, D16, D17: GREEN, SparkFun-LED:LED-1206
- added J6: (no value), SparkFun-Connectors:2X5
- added J7, J9: (no value), SparkFun-Connectors:1X12
- added JP4: (no value), adafruit:1X09-BIG
- added U$3: DRILL_SWITCH, Switch drill:DRILL_SWITCH
- IC1: value 7805T -> 74LS595D; device linear:TO220H -> 74xx-us:SO16
- J2: value 455-1750-1-ND -> 2X6; device SparkFun-Connectors:1X03 -> SparkFun-Connectors:2X6
- J3: value (none) -> 455-1750-1-ND; device SparkFun-Connectors:2X5 -> SparkFun-Connectors:1X03
- JP1, JP2, JP3: device pinhead:1X06 -> adafruit:1X09-BIG
- R1: value 100 -> 10k; device eagle-ltspice:0204/7 -> eagle-ltspice:R1206
- R2: value 330 -> 100; device eagle-ltspice:0204/7 -> eagle-ltspice:R1206
- R3, R4, R5, R6, R7, R8, R9: value 330 -> 10k; device eagle-ltspice:R1206 -> resistor:M1206
- U$8: value (none) -> DRILL_SWITCH; device StepDown_ 3.3V_D24V10F3:STEPDOWN_D24V10F3 -> Switch drill:DRILL_SWITCH
- moved JP3 644.6 mm to (-184.2, -402.6)
- moved JP2 643.0 mm to (-184.2, -397.5)
- moved JP1 641.9 mm to (-184.2, -392.4)
- moved R11 608.0 mm to (-190.5, -367.0)
- moved R10 604.4 mm to (-190.5, -361.9)
- moved U$8 578.8 mm to (-189.2, -383.5)
- moved R9 571.6 mm to (-191.8, -351.8)
- moved R8 561.5 mm to (-191.8, -341.6)
- moved R7 551.6 mm to (-191.8, -331.5)
- moved R6 541.6 mm to (-191.8, -321.3)
- moved R5 531.7 mm to (-191.8, -311.1)
- moved R4 521.9 mm to (-191.8, -301.0)
- moved R3 512.2 mm to (-191.8, -290.8)
- moved R2 458.9 mm to (-191.8, -212.1)
- moved R1 452.4 mm to (-180.3, -205.7)
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Connections:
- removed net ALERT1: B1.10, SV1.5
- removed net ALERT2: B1.11, SV2.5
- removed net ALERT3: B1.12, SV3.5
- removed net DISPLAY_DC: B1.39, DISPLAY1.DC
- removed net DISPLAY_SS: B1.38, DISPLAY1.CS
- removed net GATE: B1.43, R15.2
- removed net HC-05_ENABLE: B1.42, U$16.EN
- removed net HC-05_RX: B1.19, U$16.RX
- removed net HC-05_TX: B1.18, U$16.TX
- removed net LED8: B1.37, R12.2
- removed net MOT1_1: JP1.6, U$9.INMOT1
- removed net MOT1_2: JP1.5, U$9.INMOT2
- removed net MOT1_ENC_A: B1.A8, JP1.2
- removed net MOT1_ENC_B: B1.A9, JP1.1
- removed net MOT1_INA: B1.22, U$9.INA
- removed net MOT1_INB: B1.23, U$9.INB
- removed net MOT1_PWM: B1.2, U$9.PWM
- removed net MOT2_1: JP2.6, U$10.INMOT1
- removed net MOT2_2: JP2.5, U$10.INMOT2
- removed net MOT2_ENC_A: B1.A10, JP2.2
- removed net MOT2_ENC_B: B1.A11, JP2.1
- removed net MOT2_INA: B1.24, U$10.INA
- removed net MOT2_INB: B1.25, U$10.INB
- removed net MOT2_PWM: B1.3, U$10.PWM
- removed net MOT3_1: JP3.6, U$11.INMOT1
- removed net MOT3_2: JP3.5, U$11.INMOT2
- removed net MOT3_ENC_A: B1.A12, JP3.2
- removed net MOT3_ENC_B: B1.A13, JP3.1
- removed net MOT3_INA: B1.26, U$11.INA
- removed net MOT3_INB: B1.27, U$11.INB
- removed net MOT3_PWM: B1.4, U$11.PWM
- removed net MOT4_1: U$14.INMOT1
- removed net MOT4_2: U$14.INMOT2
- removed net MOT4_INA: B1.28, U$14.INA
- removed net MOT4_INB: B1.29, U$14.INB
- removed net MOT4_PWM: B1.5, U$14.PWM
- removed net N$10: C3.1, D2.C, U$8.VIN
- removed net N$11: LED8.A, R1.2
- removed net N$13: LED9.A, R4.1
- removed net N$14: LED10.A, R3.1
- removed net N$15: LED11.A, R5.1
- removed net N$16: LED12.A, R6.1
- removed net N$17: LED13.A, R7.1
- removed net N$18: LED14.A, R8.1
- removed net N$19: D3.C, J2.1, R13.1
- removed net N$20: D3.A, R15.1
- removed net N$23: LED1.A, R9.1
- removed net N$24: LED2.A, R12.1
- removed net N$25: R14.2, SW2.E
- removed net N$9: LED7.A, R2.2
- removed net NFC_IRQ: B1.14, M1.IRQ
- removed net NFC_SS: B1.41, M1.SS
- removed net RESET: B1.RESET, M1.RST
- removed net R_ENC_A: B1.A14, C7.2, SW2.A
- removed net R_ENC_B: B1.A15, C8.2, SW2.B
- removed net R_SEL: B1.40, R14.1
- new net INB2: U$5.INB
- new net INB3: U$6.INB
- new net KICK: B2.26, R2.2
- new net N$2: J9.3
- new net N$3: J9.4
- new net N$4: D2.C, J3.1, R1.1
- new net N$5: D2.A, R2.1
- new net N$8: J7.10
- new net P1: B2.A0, J2.1
- new net P2: B2.A1, J2.3
- new net P3: B2.A2, J2.5
- new net P4: B2.A3, J2.7
- new net P5: B2.A4, J2.9
- new net P6: B2.A5, J2.2
- new net PC1: B2.A6, J2.4
- new net PC2: B2.A7, J2.6
- new net PC3: B2.A14, J2.8
- net 12V: now also J9.10, J9.9, X3.1; no longer C1.1, D1.A, D1.C, D2.A, IC1.1, R20.1, X1.1, X4.1
- net 3.3V: now also IC1.10, IC1.15; no longer B1.3.3V, B2.3.3V, C4.1, DISPLAY1.LED, DISPLAY1.RST, DISPLAY1.VCC, IC3.10, IC3.15, M1.3V3, R1.1, U$10.VDD, U$11.VDD, U$14.VDD, U$8.VOUT, U$9.VDD
- net 5V: now also J2.11, J2.12, J6.2, J7.4, JP4.1, JP4.2, JP4.3, JP4.4, JP4.5, JP4.6, JP4.7, JP4.8, JP4.9; no longer B1.5V@0, B1.5V@1, B1.5V@2, C2.1, IC1.3, J3.2, JP1.3, JP2.3, JP3.3, R2.1, SV1.6, SV2.3, SV2.6, SV3.6, U$15.VIN, U$16.5V
- net BATTERY_LEVEL: now also B2.A15; no longer B1.A2, R20.2, R21.1
- net CLOCK: now also IC1.11; no longer IC3.11
- net DATA-OUT: now also IC1.14; no longer IC3.14
- net DRAIN: now also J3.2, X2.2; no longer J2.2, X4.2
- net ENC-A1: now also J7.5
- net ENC-A2: now also J7.11
- net ENC-A3: now also J9.5
- net ENC-B1: now also J7.6
- net ENC-B2: now also J7.12
- net ENC-B3: now also J9.6
- net GND: now also IC1.13, IC1.8, J2.10, J3.3, J6.10, J6.6, J6.8, J7.3, J9.11, J9.12, JP1.1, JP1.2, JP1.3, JP1.5, JP1.6, JP1.7, JP1.8, JP1.9, R1.2, R3.1, R4.1, R5.1, R6.1, R7.1, R8.1, R9.1, X4.2; no longer B1.GND@0, B1.GND@1, B1.GND@2, B1.GND@3, B1.GND@4, C1.2, C2.2, C3.2, C4.2, C7.1, C8.1, DISPLAY1.GND, IC1.2, IC3.13, IC3.8, J2.3, J3.10, J3.6, J3.8, JP2.4, JP3.4, LED1.K, LED10.K, LED11.K, LED12.K, LED13.K, LED14.K, LED2.K, LED7.K, LED8.K, LED9.K, M1.GND, R13.2, R21.2, RN1.1, SV1.1, SV1.3, SV2.1, SV3.1, SW2.C, SW2.D, U$10.GND, U$10.GND2, U$10.GNDMOT-1, U$11.GND, U$11.GND2, U$11.GNDMOT-1, U$14.GND, U$14.GND2, U$14.GNDMOT-1, U$15.GND, U$16.GND, U$8.GND, U$9.GND, U$9.GND2, U$9.GNDMOT-1, X1.2, X2.2, X5.2
- net LATCH: now also IC1.12; no longer IC3.12
- net LED1: now also D11.A, D11.C, IC1.1, R3.2; no longer B1.30, IC3.1, R4.2, RN1.2
- net LED2: now also D12.A, D12.C, IC1.2, R4.2; no longer B1.31, IC3.2, R3.2, RN1.3
- net LED3: now also D13.A, D13.C, IC1.3; no longer B1.32, IC3.3, RN1.4
- net LED4: now also D14.A, D14.C, IC1.4; no longer B1.33, IC3.4, RN1.5
- net LED5: now also D15.A, D15.C, IC1.5; no longer B1.34, IC3.5, RN1.6
- net LED6: now also D16.A, D16.C, IC1.6; no longer B1.35, IC3.6, RN1.7
- net LED7: now also D17.A, D17.C, IC1.7; no longer B1.36, IC3.7, RN1.8
- net MISO: now also B2.50, J6.1; no longer B1.50, J3.1, M1.MISO
- net MOSI: now also B2.51, J6.4; no longer B1.51, DISPLAY1.SDA, J3.4, M1.MOSI
- net MOTA1: now also J7.1
- net MOTA2: now also J7.7
- net MOTA3: now also J9.1
- net MOTB1: now also J7.2
- net MOTB2: now also J7.8
- net MOTB3: now also J9.2
- net N$7: now also J7.9; no longer B2.26
- net PIXY_SS: now also B2.53, J6.7; no longer B1.53, J3.7
- net ROLLERA: now also J9.7
- net ROLLERB: now also J9.8
- net SCK: now also B2.52, J6.3; no longer B1.52, DISPLAY1.SCK, J3.3, M1.SCK
- net SCL: now also J6.5, JP3.1, JP3.2, JP3.3, JP3.4, JP3.5, JP3.6, JP3.7, JP3.8, JP3.9; no longer B1.21, J3.5, SV1.2, SV2.2, SV3.2, U$15.SCL
- net SDA: now also J6.9, JP2.1, JP2.2, JP2.3, JP2.4, JP2.5, JP2.6, JP2.7, JP2.8, JP2.9; no longer B1.20, J3.9, SV1.4, SV2.4, SV3.3, SV3.4, U$15.SDA
- net VCC: now also IC1.16; no longer IC3.16
- net VMOT: now also X4.1; no longer U$10.VMOT-1, U$11.VMOT-1, U$14.VMOT-1, U$9.VMOT-1, X3.1, X5.1
Other:
- board size 100 x 80 mm -> 193 x 168.9 mm
