File: elettronica/sensori di liena.sch (EAGLE design)
At the start: 17 parts, among them J2 2X6, T1 BP103

Commit message: continuare a posizionare i pezzi nella board
Parts:
- added C1: 0.1uF, SparkFun-Capacitors:0.1UF-KIT-EZ-50V-20%
- added D2: 1N4148, diode:1N4148DO35-7
- added J3: 455-1750-1-ND, SparkFun-Connectors:CONN_03
- added R3: 10k, eagle-ltspice:RR1206
- added R4: 100, eagle-ltspice:RR1206
- added X2: (no value), con-ptr500:AK500/2-H
Connections:
- new net DRAIN: J3.2, X2-2.KL
- new net KICK: R4.2
- new net N$4: D2.C, J3.1, R3.1
- new net N$5: D2.A, R4.1
- net 12V: now also X2-1.KL
- net GND: now also C1.2, J3.3, JP1.3, R3.2
- net GND-PT: no longer JP1.3
- net PT1: now also C1.1
Other:
- note added: "Solenoid"
- note added: "stp16nf06"
Changed lines of the file:
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@@
 <?xml version="1.0" encoding="utf-8"?>
 <!DOCTYPE eagle SYSTEM "eagle.dtd">
-<eagle version="9.3.0">
+<eagle version="9.2.2">
 <drawing>
 <settings>
@@
 <part name="J9" library="SparkFun-Connectors" library_urn="urn:adsk.eagle:library:513" deviceset="CONN_12" device="" package3d_urn="urn:adsk.eagle:package:38169/1"/>
 <part name="J7" library="SparkFun-Connectors" library_urn="urn:adsk.eagle:library:513" deviceset="CONN_12" device="" package3d_urn="urn:adsk.eagle:package:38169/1"/>
+<part name="C1" library="SparkFun-Capacitors" library_urn="urn:adsk.eagle:library:510" deviceset="0.1UF" device="-KIT-EZ-50V-20%" package3d_urn="urn:adsk.eagle:package:37428/1" value="0.1uF"/>
+<part name="J3" library="SparkFun-Connectors" deviceset="CONN_03" device="" value="455-1750-1-ND"/>
+<part name="X2" library="con-ptr500" library_urn="urn:adsk.eagle:library:181" deviceset="AK500/2-H" device="" package3d_urn="urn:adsk.eagle:package:9901/1"/>
+<part name="D2" library="diode" library_urn="urn:adsk.eagle:library:210" deviceset="1N4148" device="DO35-7" package3d_urn="urn:adsk.eagle:package:43339/1" value="1N4148"/>
+<part name="R3" library="eagle-ltspice" library_urn="urn:adsk.eagle:library:217" deviceset="R" device="R1206" package3d_urn="urn:adsk.eagle:package:13301/1" value="10k"/>
+<part name="R4" library="eagle-ltspice" library_urn="urn:adsk.eagle:library:217" deviceset="R" device="R1206" package3d_urn="urn:adsk.eagle:package:13301/1" value="100"/>
 </parts>
 <sheets>
@@
 <wire x1="256.54" y1="25.4" x2="256.54" y2="175.26" width="1.016" layer="97" style="longdash"/>
 <wire x1="256.54" y1="175.26" x2="96.52" y2="175.26" width="1.016" layer="97" style="longdash"/>
-<wire x1="96.52" y1="175.26" x2="96.52" y2="71.12" width="1.016" layer="97" style="longdash"/>
+<wire x1="96.52" y1="175.26" x2="96.52" y2="127" width="1.016" layer="97" style="longdash"/>
 <text x="30.48" y="167.64" size="5.08" layer="97">Sensors hub</text>
+<wire x1="96.52" y1="127" x2="96.52" y2="71.12" width="1.016" layer="97" style="longdash"/>
 <wire x1="5.08" y1="71.12" x2="96.52" y2="71.12" width="1.016" layer="97" style="longdash"/>
 <wire x1="5.08" y1="27.94" x2="60.96" y2="27.94" width="1.016" layer="97" style="longdash"/>
 <text x="10.16" y="63.5" size="3.81" layer="97">peripheral sensors</text>
 <wire x1="60.96" y1="27.94" x2="60.96" y2="71.12" width="1.016" layer="97" style="longdash"/>
-<text x="33.02" y="35.56" size="2.54" layer="97">Total of 6</text>
+<text x="43.18" y="35.56" size="2.54" layer="97">Total of 6</text>
 <wire x1="5.08" y1="175.26" x2="5.08" y2="71.12" width="1.016" layer="97" style="longdash"/>
 <wire x1="5.08" y1="175.26" x2="96.52" y2="175.26" width="1.016" layer="97" style="longdash"/>
@@
 <wire x1="5.08" y1="5.334" x2="5.08" y2="71.12" width="1.016" layer="97" style="longdash"/>
 <text x="110.998" y="166.878" size="5.08" layer="97">Motor hub</text>
+<wire x1="96.52" y1="127" x2="157.48" y2="127" width="1.016" layer="97" style="longdash"/>
+<wire x1="157.48" y1="127" x2="157.48" y2="172.72" width="1.016" layer="97" style="longdash"/>
+<text x="101.6" y="121.92" size="1.778" layer="97">stp16nf06</text>
+<text x="118.364" y="120.396" size="2.54" layer="97">Solenoid</text>
 </plain>
 <instances>
@@
 <attribute name="VALUE" x="127" y="167.386" size="1.778" layer="96" font="vector" rot="R180"/>
 <attribute name="NAME" x="127" y="131.572" size="1.778" layer="95" font="vector" rot="R180"/>
+</instance>
+<instance part="C1" gate="G$1" x="27.94" y="33.02" smashed="yes">
+<attribute name="NAME" x="30.48" y="33.655" size="1.778" layer="95" font="vector"/>
+<attribute name="VALUE" x="33.274" y="33.401" size="1.778" layer="96" font="vector"/>
+</instance>
+<instance part="J3" gate="J$1" x="106.68" y="114.3" smashed="yes">
+<attribute name="NAME" x="104.14" y="119.888" size="1.778" layer="95" font="vector"/>
+</instance>
+<instance part="X2" gate="-1" x="106.68" y="99.06" smashed="yes">
+<attribute name="NAME" x="105.41" y="99.949" size="1.778" layer="95" rot="R180"/>
+</instance>
+<instance part="X2" gate="-2" x="106.68" y="93.98" smashed="yes">
+<attribute name="NAME" x="105.41" y="94.869" size="1.778" layer="95" rot="R180"/>
+<attribute name="VALUE" x="102.87" y="90.297" size="1.778" layer="96"/>
+</instance>
+<instance part="D2" gate="G$1" x="124.46" y="111.76" smashed="yes" rot="R180">
+<attribute name="NAME" x="129.54" y="113.8174" size="1.778" layer="95" rot="R180"/>
+</instance>
+<instance part="R3" gate="G$1" x="127" y="106.68" smashed="yes">
+<attribute name="NAME" x="125.73" y="108.1786" size="1.778" layer="95"/>
+<attribute name="VALUE" x="123.19" y="103.378" size="1.778" layer="96"/>
+</instance>
+<instance part="R4" gate="G$1" x="134.62" y="111.76" smashed="yes">
+<attribute name="NAME" x="133.35" y="113.2586" size="1.778" layer="95"/>
+<attribute name="VALUE" x="130.81" y="108.458" size="1.778" layer="96"/>
 </instance>
 </instances>
@@
 <wire x1="142.24" y1="137.16" x2="142.24" y2="134.62" width="0.1524" layer="91"/>
 <label x="142.24" y="134.62" size="1.016" layer="95" xref="yes"/>
+</segment>
+<segment>
+<pinref part="JP1" gate="A" pin="3"/>
+<pinref part="C1" gate="G$1" pin="2"/>
+<wire x1="12.7" y1="33.02" x2="22.86" y2="33.02" width="0.1524" layer="91"/>
+<wire x1="22.86" y1="33.02" x2="27.94" y2="30.48" width="0.1524" layer="91"/>
+<label x="27.94" y="30.48" size="1.27" layer="95" xref="yes"/>
+</segment>
+<segment>
+<pinref part="J3" gate="J$1" pin="3"/>
+<wire x1="114.3" y1="116.84" x2="116.84" y2="116.84" width="0.1524" layer="91" style="longdash"/>
+<label x="116.84" y="116.84" size="1.27" layer="95" xref="yes"/>
+</segment>
+<segment>
+<pinref part="R3" gate="G$1" pin="2"/>
+<wire x1="132.08" y1="106.68" x2="134.62" y2="106.68" width="0.1524" layer="91"/>
+<label x="134.62" y="106.68" size="1.27" layer="95" xref="yes"/>
 </segment>
 </net>
@@
 <segment>
 <pinref part="JP1" gate="A" pin="1"/>
-<wire x1="12.7" y1="38.1" x2="17.78" y2="38.1" width="0.1524" layer="91"/>
-<label x="17.78" y="38.1" size="1.27" layer="95" xref="yes"/>
+<wire x1="12.7" y1="38.1" x2="27.94" y2="38.1" width="0.1524" layer="91"/>
+<label x="27.94" y="38.1" size="1.27" layer="95" xref="yes"/>
+<pinref part="C1" gate="G$1" pin="1"/>
 </segment>
 </net>
 <net name="GND-PT" class="0">
-<segment>
-<pinref part="JP1" gate="A" pin="3"/>
-<wire x1="12.7" y1="33.02" x2="17.78" y2="33.02" width="0.1524" layer="91"/>
-<label x="17.78" y="33.02" size="1.27" layer="95" xref="yes"/>
-</segment>
 <segment>
 <pinref part="R1" gate="G$1" pin="2"/>
@@
 <label x="142.24" y="139.7" size="1.016" layer="95" xref="yes"/>
 </segment>
+<segment>
+<pinref part="X2" gate="-1" pin="KL"/>
+<wire x1="111.76" y1="99.06" x2="114.3" y2="99.06" width="0.1524" layer="91" style="longdash"/>
+<label x="114.3" y="99.06" size="1.27" layer="95" xref="yes"/>
+</segment>
 </net>
 <net name="ENC-A1" class="0">
@@
 </segment>
 </net>
+<net name="KICK" class="0">
+<segment>
+<pinref part="R4" gate="G$1" pin="2"/>
+<wire x1="139.7" y1="111.76" x2="142.24" y2="111.76" width="0.1524" layer="91" style="longdash"/>
+<label x="142.24" y="111.76" size="1.27" layer="95" xref="yes"/>
+</segment>
+</net>
+<net name="DRAIN" class="0">
+<segment>
+<pinref part="J3" gate="J$1" pin="2"/>
+<wire x1="114.3" y1="114.3" x2="116.84" y2="114.3" width="0.1524" layer="91" style="longdash"/>
+<label x="116.84" y="114.3" size="1.27" layer="95" xref="yes"/>
+</segment>
+<segment>
+<pinref part="X2" gate="-2" pin="KL"/>
+<wire x1="111.76" y1="93.98" x2="114.3" y2="93.98" width="0.1524" layer="91" style="longdash"/>
+<label x="114.3" y="93.98" size="1.27" layer="95" xref="yes"/>
+</segment>
+</net>
+<net name="N$4" class="0">
+<segment>
+<pinref part="D2" gate="G$1" pin="C"/>
+<pinref part="J3" gate="J$1" pin="1"/>
+<wire x1="121.92" y1="111.76" x2="116.84" y2="111.76" width="0.1524" layer="91"/>
+<junction x="116.84" y="111.76"/>
+<wire x1="116.84" y1="111.76" x2="114.3" y2="111.76" width="0.1524" layer="91"/>
+<wire x1="116.84" y1="111.76" x2="116.84" y2="106.68" width="0.1524" layer="91"/>
+<pinref part="R3" gate="G$1" pin="1"/>
+<wire x1="121.92" y1="106.68" x2="116.84" y2="106.68" width="0.1524" layer="91"/>
+</segment>
+</net>
+<net name="N$5" class="0">
+<segment>
+<pinref part="D2" gate="G$1" pin="A"/>
+<wire x1="127" y1="111.76" x2="129.54" y2="111.76" width="0.1524" layer="91" style="longdash"/>
+<pinref part="R4" gate="G$1" pin="1"/>
+</segment>
+</net>

Commit message: sensori di linea done
Parts:
- removed D2: 1N4148, diode:1N4148DO35-7
- removed J2: 2X6, SparkFun-Connectors:CONN_06X2PTH_FEMALE
- removed J3: 455-1750-1-ND, SparkFun-Connectors:CONN_03
- removed J7, J9: (no value), SparkFun-Connectors:CONN_12
- removed JP10, JP11, JP3, JP4, JP5, JP6, JP7, JP8, JP9: (no value), pinhead:PINHD-1X3
- removed R1: 10k, eagle-ltspice:R0204/7
- removed R3: 10k, eagle-ltspice:RR1206
- removed X2: (no value), con-ptr500:AK500/2-H
- R2: value 100 -> 10k; device eagle-ltspice:R0204/7 -> SparkFun-Resistors:10KOHM-0603-1/10W-1%
- R4: device eagle-ltspice:RR1206 -> SparkFun-Resistors:10KOHM-0603-1/10W-1%
Connections:
- removed net 12V: J9.10, J9.9, X2-1.KL
- removed net 5V: J2.11, J2.12, J7.4, JP10.2, JP11.2, JP3.2, JP4.2, JP5.2, JP6.2, JP7.2, JP8.2, JP9.2
- removed net DRAIN: J3.2, X2-2.KL
- removed net ENC-A1: J7.5
- removed net ENC-A2: J7.11
- removed net ENC-A3: J9.5
- removed net ENC-B1: J7.6
- removed net ENC-B2: J7.12
- removed net ENC-B3: J9.6
- removed net KICK: R4.2
- removed net MOTA1: J7.1
- removed net MOTA2: J7.7
- removed net MOTA3: J9.1
- removed net MOTB1: J7.2
- removed net MOTB2: J7.8
- removed net MOTB3: J9.2
- removed net N$3: J9.4
- removed net N$4: D2.C, J3.1, R3.1
- removed net N$5: D2.A, R4.1
- removed net N$7: J7.9
- removed net N$8: J7.10
- removed net P1: J2.1, JP3.1
- removed net P2: J2.3, JP4.1
- removed net P3: J2.5, JP5.1
- removed net P4: J2.7, JP6.1
- removed net P5: J2.9, JP7.1
- removed net P6: J2.2, JP8.1
- removed net PC1: J2.4, JP9.1
- removed net PC2: J2.6, JP10.1
- removed net PC3: J2.8, JP11.1
- removed net ROLLERA: J9.7
- removed net ROLLERB: J9.8
- net GND: no longer J2.10, J3.3, J7.3, J9.11, J9.12, JP10.3, JP11.3, JP3.3, JP4.3, JP5.3, JP6.3, JP7.3, JP8.3, JP9.3, R3.2
- net GND-PT: now also R2.1, R4.1; no longer R1.2, R2.2
- net N$2: now also R4.2; no longer J9.3, R2.1
- net PT1: now also R2.2; no longer R1.1
Other:
- note removed: "Motor hub"
- note removed: "Sensors hub"
- note removed: "Solenoid"
- note removed: "stp16nf06"
- moved on the sheet: C1, D1, JP1, T1

Commit message: pcb definitiva 2.0
Changed lines of the file:
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@@
 </variantdefs>
 <classes>
-<class number="0" name="default" width="0.254" drill="0">
+<class number="0" name="5v" width="0.508" drill="0">
 <clearance class="0" value="0.1524"/>
 </class>
@@
 <pinref part="JP1" gate="A" pin="3"/>
 <pinref part="C1" gate="G$1" pin="2"/>
-<wire x1="12.7" y1="137.16" x2="22.86" y2="137.16" width="0.1524" layer="91"/>
-<wire x1="22.86" y1="137.16" x2="27.94" y2="134.62" width="0.1524" layer="91"/>
+<wire x1="12.7" y1="137.16" x2="20.32" y2="137.16" width="0.1524" layer="91"/>
+<wire x1="20.32" y1="137.16" x2="27.94" y2="134.62" width="0.1524" layer="91"/>
 <label x="27.94" y="134.62" size="1.27" layer="95" xref="yes"/>
 </segment>
