File: elettronica/sensori di liena.brd (EAGLE design)
At the start: 160 x 100 mm, 23 parts, among them J2 2X6, J3 455-1750-1-ND, T1 BP103

Commit message: sensori di linea done
Parts:
- removed D2: 1N4148, diode:DO35-7
- removed J2: 2X6, SparkFun-Connectors:2X6
- removed J3: 455-1750-1-ND, SparkFun-Connectors:1X03
- removed J7, J9: (no value), SparkFun-Connectors:1X12
- removed JP10, JP11, JP3, JP4, JP5, JP6, JP7, JP8, JP9: (no value), pinhead:1X03
- removed R1: 10k, eagle-ltspice:0204/7
- removed R3: 10k, eagle-ltspice:R1206
- removed X2: (no value), con-ptr500:AK500/2-H
- R2: value 100 -> 10k; device eagle-ltspice:0204/7 -> SparkFun-Resistors:0603
- R4: device eagle-ltspice:R1206 -> SparkFun-Resistors:0603
- moved R4 149.7 mm to (61.0, 54.9)
- moved C1 130.9 mm to (55.4, 59.9), turned to 90 degrees
- moved R2 121.8 mm to (58.7, 57.1), turned to 180 degrees
- moved JP1 120.0 mm to (58.4, 63.2), turned to 90 degrees
- moved D1 117.8 mm to (62.5, 63.8)
- moved T1 117.3 mm to (63.8, 58.7)
Connections:
- removed net 12V: J9.10, J9.9, X2.1
- removed net 5V: J2.11, J2.12, J7.4, JP10.2, JP11.2, JP3.2, JP4.2, JP5.2, JP6.2, JP7.2, JP8.2, JP9.2
- removed net DRAIN: J3.2, X2.2
- removed net ENC-A1: J7.5
- removed net ENC-A2: J7.11
- removed net ENC-A3: J9.5
- removed net ENC-B1: J7.6
- removed net ENC-B2: J7.12
- removed net ENC-B3: J9.6
- removed net KICK: R4.2
- removed net MOTA1: J7.1
- removed net MOTA2: J7.7
- removed net MOTA3: J9.1
- removed net MOTB1: J7.2
- removed net MOTB2: J7.8
- removed net MOTB3: J9.2
- removed net N$3: J9.4
- removed net N$4: D2.C, J3.1, R3.1
- removed net N$5: D2.A, R4.1
- removed net N$7: J7.9
- removed net N$8: J7.10
- removed net P1: J2.1, JP3.1
- removed net P2: J2.3, JP4.1
- removed net P3: J2.5, JP5.1
- removed net P4: J2.7, JP6.1
- removed net P5: J2.9, JP7.1
- removed net P6: J2.2, JP8.1
- removed net PC1: J2.4, JP9.1
- removed net PC2: J2.6, JP10.1
- removed net PC3: J2.8, JP11.1
- removed net ROLLERA: J9.7
- removed net ROLLERB: J9.8
- net GND: no longer J2.10, J3.3, J7.3, J9.11, J9.12, JP10.3, JP11.3, JP3.3, JP4.3, JP5.3, JP6.3, JP7.3, JP8.3, JP9.3, R3.2
- net GND-PT: now also R2.1, R4.1; no longer R1.2, R2.2
- net N$2: now also R4.2; no longer J9.3, R2.1
- net PT1: now also R2.2; no longer R1.1
Routing:
- net N$2: track 0.00 -> 13.0 mm, vias 0 -> 1
- net PT1: track 0.00 -> 11.6 mm
- net 5V-PT: track 0.00 -> 8.65 mm
- net GND: track 0.00 -> 5.73 mm
- net GND-PT: track 0.00 -> 2.62 mm
- added copper zone on layer 1, net GND
- added copper zone on layer 16, net GND
Other:
- board size 160 x 100 mm -> 14 x 24 mm

Commit message: pcb definitiva 2.0
Routing:
- net N$2: track 13.0 -> 9.95 mm
- net 5V-PT: track 8.65 -> 9.28 mm
Changed lines of the file:
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@@
 </variantdefs>
 <classes>
-<class number="0" name="default" width="0.254" drill="0">
+<class number="0" name="5v" width="0.508" drill="0">
 <clearance class="0" value="0.1524"/>
 </class>
@@
 <contactref element="JP1" pad="3"/>
 <contactref element="C1" pad="2"/>
-<wire x1="55.4736" y1="62.7888" x2="58.3184" y2="65.6336" width="0.254" layer="1"/>
-<wire x1="55.4736" y1="61.3664" x2="55.4736" y2="62.7888" width="0.254" layer="1"/>
-<wire x1="58.3184" y1="65.6336" x2="58.42" y2="65.786" width="0.254" layer="1"/>
-<wire x1="55.4736" y1="61.3664" x2="55.372" y2="61.341" width="0.254" layer="1"/>
+<wire x1="55.4736" y1="62.9412" x2="58.3184" y2="65.786" width="0.508" layer="1"/>
+<wire x1="55.4736" y1="61.5188" x2="55.4736" y2="62.9412" width="0.508" layer="1"/>
+<wire x1="58.3184" y1="65.786" x2="58.42" y2="65.786" width="0.508" layer="1"/>
+<wire x1="55.4736" y1="61.5188" x2="55.372" y2="61.341" width="0.508" layer="1"/>
+<polygon width="0.254" layer="1" isolate="0.3048">
+<vertex x="40.894" y="78.232"/>
+<vertex x="40.894" y="43.434"/>
+<vertex x="83.058" y="43.434"/>
+<vertex x="83.058" y="78.232"/>
+</polygon>
 <polygon width="0.254" layer="16" isolate="0.3048">
-<vertex x="48.514" y="73.66"/>
-<vertex x="48.514" y="44.958"/>
-<vertex x="71.628" y="44.958"/>
-<vertex x="71.628" y="73.66"/>
-</polygon>
-<polygon width="0.254" layer="1">
-<vertex x="48.514" y="73.914"/>
-<vertex x="48.514" y="46.736"/>
-<vertex x="73.152" y="46.736"/>
-<vertex x="73.152" y="73.914"/>
+<vertex x="45.974" y="74.93"/>
+<vertex x="45.974" y="46.228"/>
+<vertex x="74.93" y="46.228"/>
+<vertex x="74.93" y="74.93"/>
 </polygon>
 </signal>
@@
 <contactref element="C1" pad="1"/>
 <contactref element="R2" pad="2"/>
-<wire x1="56.6928" y1="57.3024" x2="57.7088" y2="57.3024" width="0.254" layer="1"/>
-<wire x1="55.4736" y1="58.5216" x2="56.6928" y2="57.3024" width="0.254" layer="1"/>
-<wire x1="57.7088" y1="57.3024" x2="57.824" y2="57.15" width="0.254" layer="1"/>
-<wire x1="55.4736" y1="58.5216" x2="55.372" y2="58.547" width="0.254" layer="1"/>
-<wire x1="61.3664" y1="57.7088" x2="62.5856" y2="57.7088" width="0.254" layer="1"/>
-<wire x1="58.5216" y1="60.5536" x2="59.7408" y2="59.3344" width="0.254" layer="1"/>
-<wire x1="59.7408" y1="59.3344" x2="61.3664" y2="57.7088" width="0.254" layer="1"/>
-<wire x1="62.5856" y1="57.7088" x2="62.738" y2="57.658" width="0.254" layer="1"/>
-<wire x1="58.5216" y1="60.5536" x2="58.42" y2="60.706" width="0.254" layer="1"/>
-<wire x1="59.7408" y1="59.1312" x2="57.912" y2="57.3024" width="0.254" layer="1"/>
-<wire x1="59.7408" y1="59.3344" x2="59.7408" y2="59.1312" width="0.254" layer="1"/>
-<wire x1="57.912" y1="57.3024" x2="57.824" y2="57.15" width="0.254" layer="1"/>
+<wire x1="56.5404" y1="57.2516" x2="57.6072" y2="57.2516" width="0.508" layer="1"/>
+<wire x1="55.4736" y1="58.3184" x2="56.5404" y2="57.2516" width="0.508" layer="1"/>
+<wire x1="57.6072" y1="57.2516" x2="57.824" y2="57.15" width="0.508" layer="1"/>
+<wire x1="55.4736" y1="58.3184" x2="55.372" y2="58.547" width="0.508" layer="1"/>
+<wire x1="61.1632" y1="57.9628" x2="62.5856" y2="57.9628" width="0.508" layer="1"/>
+<wire x1="58.42" y1="60.706" x2="59.563" y2="59.563" width="0.508" layer="1"/>
+<wire x1="59.563" y1="59.563" x2="61.1632" y2="57.9628" width="0.508" layer="1"/>
+<wire x1="62.5856" y1="57.9628" x2="62.738" y2="57.658" width="0.508" layer="1"/>
+<wire x1="57.9628" y1="57.9628" x2="57.9628" y2="57.2516" width="0.508" layer="1"/>
+<wire x1="59.563" y1="59.563" x2="57.9628" y2="57.9628" width="0.508" layer="1"/>
+<wire x1="57.9628" y1="57.2516" x2="57.824" y2="57.15" width="0.508" layer="1"/>
 </signal>
 <signal name="GND-PT">
 <contactref element="R2" pad="1"/>
 <contactref element="R4" pad="1"/>
-<wire x1="59.5376" y1="55.2704" x2="59.5376" y2="57.0992" width="0.254" layer="1"/>
-<wire x1="59.944" y1="54.864" x2="59.5376" y2="55.2704" width="0.254" layer="1"/>
-<wire x1="59.5376" y1="57.0992" x2="59.524" y2="57.15" width="0.254" layer="1"/>
-<wire x1="59.944" y1="54.864" x2="60.11" y2="54.864" width="0.254" layer="1"/>
+<wire x1="59.7408" y1="55.4736" x2="59.7408" y2="56.896" width="0.508" layer="1"/>
+<wire x1="60.0964" y1="55.118" x2="59.7408" y2="55.4736" width="0.508" layer="1"/>
+<wire x1="59.7408" y1="56.896" x2="59.524" y2="57.15" width="0.508" layer="1"/>
+<wire x1="60.0964" y1="55.118" x2="60.11" y2="54.864" width="0.508" layer="1"/>
 </signal>
 <signal name="5V-PT">
@@
 <contactref element="T1" pad="C"/>
 <contactref element="D1" pad="A"/>
-<wire x1="64.6176" y1="60.3504" x2="64.6176" y2="59.7408" width="0.254" layer="1"/>
-<wire x1="61.214" y1="63.754" x2="64.6176" y2="60.3504" width="0.254" layer="1"/>
-<wire x1="64.6176" y1="59.7408" x2="64.77" y2="59.69" width="0.254" layer="1"/>
-<wire x1="60.96" y1="63.3984" x2="58.5216" y2="63.3984" width="0.254" layer="1"/>
-<wire x1="61.1632" y1="63.6016" x2="60.96" y2="63.3984" width="0.254" layer="1"/>
-<wire x1="58.5216" y1="63.3984" x2="58.42" y2="63.246" width="0.254" layer="1"/>
-<wire x1="61.1632" y1="63.6016" x2="61.214" y2="63.754" width="0.254" layer="1"/>
+<wire x1="64.7192" y1="60.452" x2="64.7192" y2="59.7408" width="0.508" layer="1"/>
+<wire x1="61.5188" y1="63.6524" x2="64.7192" y2="60.452" width="0.508" layer="1"/>
+<wire x1="64.7192" y1="59.7408" x2="64.77" y2="59.69" width="0.508" layer="1"/>
+<wire x1="61.5188" y1="63.6524" x2="61.214" y2="63.754" width="0.508" layer="1"/>
+<wire x1="61.5188" y1="63.2968" x2="58.674" y2="63.2968" width="0.508" layer="1"/>
+<wire x1="58.674" y1="63.2968" x2="58.42" y2="63.246" width="0.508" layer="1"/>
+<wire x1="61.5188" y1="63.2968" x2="61.214" y2="63.754" width="0.508" layer="1"/>
 </signal>
 <signal name="N$2">
 <contactref element="D1" pad="K"/>
 <contactref element="R4" pad="2"/>
-<wire x1="61.81" y1="54.864" x2="63.472434375" y2="54.864" width="0.254" layer="1"/>
-<wire x1="63.472434375" y1="54.864" x2="63.5718875" y2="54.764546875" width="0.254" layer="1"/>
-<via x="63.5718875" y="54.764546875" extent="1-16" drill="0.508"/>
-<wire x1="63.5718875" y1="54.764546875" x2="61.214" y2="57.122434375" width="0.254" layer="16"/>
-<wire x1="61.214" y1="60.452" x2="64.008" y2="63.246" width="0.254" layer="16"/>
-<wire x1="64.008" y1="63.246" x2="64.008" y2="63.5" width="0.254" layer="16"/>
-<wire x1="64.008" y1="63.5" x2="63.754" y2="63.754" width="0.254" layer="16"/>
-<wire x1="61.214" y1="57.122434375" x2="61.214" y2="60.452" width="0.254" layer="16"/>
+<wire x1="61.5188" y1="56.5404" x2="61.5188" y2="55.118" width="0.508" layer="1"/>
+<wire x1="61.5188" y1="61.5188" x2="61.5188" y2="56.5404" width="0.508" layer="16"/>
+<wire x1="63.754" y1="63.754" x2="61.5188" y2="61.5188" width="0.508" layer="16"/>
+<wire x1="61.5188" y1="55.118" x2="61.81" y2="54.864" width="0.508" layer="1"/>
+<via x="61.5188" y="56.5404" extent="1-16" drill="0.508"/>
 </signal>
 </signals>
